File: SAS_PCBv2/power.kicad_sch (KiCad schematic)
At the start: 18 parts, among them J3 Conn_01x02_Pin, Q2 2N4403, Q3 2N4403, SW1 SW_SPST, U2 LF33_TO220

Commit message: Ajout du connecteur spécial pour les radios, insertion des footprints dans le PCB, fin du schéma
Parts:
- C1: footprint (none) -> SAS_PCBv2_footprint:CAP_RR71_NIC
- C11, C2: footprint (none) -> Capacitor_THT:CP_Radial_D5.0mm_P2.00mm; Digikey (none) -> 1189-2322-ND
- C14, C15: footprint (none) -> Capacitor_THT:CP_Radial_D5.0mm_P2.00mm
- C16: footprint (none) -> SAS_PCBv2_footprint:CAP_C320_KEM
- R10: footprint (none) -> Resistor_THT:R_Axial_DIN0207_L6.3mm_D2.5mm_P10.16mm_Horizontal; Digikey (none) -> MFR-25FRF52-10K
- R11: footprint (none) -> Resistor_THT:R_Axial_DIN0207_L6.3mm_D2.5mm_P10.16mm_Horizontal; Digikey (none) -> MFR-25FRF52-47K
