File: SAS_PCBv2/SAS_PCBv2.kicad_sch (KiCad schematic)
At the start: 1 part, among them J2 Raspberry Pi 4 Model B

Commit message: Fix footprints, widen power traces, route RPi cables, fix transistor pinout
Other:
- note added: "Cables : 600AC0001 + 600AB0001(5V / 3A)"
Changed lines of the file:
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@@
 	(generator_version "10.0")
 	(paper "A4")
+	(text "Cables : 600AC0001 + 600AB0001(5V / 3A)"
+		(exclude_from_sim no)
+		(at 178.562 148.844 0)
+		(effects
+			(font
+				(size 1.27 1.27)
+			)
+		)
+	)
 	(junction
 		(at 198.12 96.52)
