File: SAS_PCBv2/SAS_PCBv2.kicad_pcb (KiCad board)
At the start: 2 copper layers, 108 x 78 mm, 56 parts, among them J1 GY-BMP280, J10 Conn_01x04, J11 Conn_01x04, J12 GY-GPS6MV2, J14 Fan PWM, J16 GT17HN-4DP-2HD56, J17 GT17HN-4DP-2HD56, J2 Raspberry Pi 4 Model B, J3 Conn_01x02_Pin, J4 Conn_01x02, J5 Conn_01x02, J6 Conn_01x02, J7 Conn_01x02, J8 Conn_01x02, J9 Conn_01x02, Q2 2N4403, Q3 2N4403, Q4 BS170, Q5 BS170, SW2 SW_SPDT, U2 LF33_TO220

Commit message: finition et fabrication
Parts:
- added G***: LOGO, LOGO, B.Cu at (170.3, 76.7)
- G***: moved to B.Cu
- J3: footprint Connector_PinHeader_2.54mm:PinHeader_1x02_P2.54mm_Vertical -> Connector_AMASS:AMASS_XT30U-M_1x02_P5.0mm_Vertical
- moved G*** 59.8 mm to (201.7, 91.1), turned to 180 degrees
- moved J3 1.53 mm to (134.7, 58.8), turned to 90 degrees
Connections:
- F1 pad 1: Net-(J3-Pin_1) -> Net-(J3-Pin_2)
- J3 pad 1: Net-(J3-Pin_1) -> GND
- J3 pad 2: GND -> Net-(J3-Pin_2)
Routing:
- net GND: track 99.9 -> 43.7 mm, vias 1 -> 2
- net Net-(J3-Pin_2): track 0.00 -> 11.4 mm
- net Net-(J3-Pin_1): track 9.10 -> 0.00 mm
- net BTN_5: track 98.1 -> 102.5 mm
- net BTN_6: track 108.6 -> 112.5 mm
- net UART_GPS_RX: track 79.1 -> 75.9 mm
- net UART_RAD2_RX: track 77.6 -> 80.1 mm
- net UART_GPS_TX: track 87.3 -> 85.4 mm
- net BTN_4: track 87.5 -> 89.3 mm
- net RPI_5V: track 42.9 -> 41.6 mm
- net Vent_PWM: track 71.9 -> 72.7 mm
- net UART_RAD1_RX: track 83.5 -> 82.9 mm
- added copper zone on F.Cu, net GND
Other:
- board text added: "ABRARACOURCIX le chef du village!"
- board text added: "BARO"
- board text added: "BTN1"
- board text added: "BTN2"
- board text added: "BTN3"
- board text added: "BTN4"
- board text added: "BTN5"
- board text added: "BTN6"
- board text added: "GPS"
- board text added: "LCD"
- board text added: "Louis-Charles Blais Édouard Bélanger SAS PCB v2.0 07-2026"
- board text added: "RFD1"
- board text added: "RFD2"
- board text added: "RPI"
- board text added: "TACH"
- board text added: "Vin"
